File: kicad/buspirate-breadboard-connector.kicad_pcb (KiCad board)
At the start: 2 copper layers, 17.8 x 15.2 mm, 2 parts

Commit message: minor changes to the footprints and creation of gerbers
Parts:
- BP1: footprint Pin_Headers:Pin_Header_Straight_2x05 -> breadboard-connector:header_2x5
Other:
- net class Default: clearance 0.2 -> 0.1524; trace_width 0.25 -> 0.1524; via_dia 0.6 -> 0.6858; via_drill 0.4 -> 0.3302
- rule trace_clearance: 0.2 -> 0.1524
- rule trace_min: 0.2 -> 0.1524
- rule via_min_drill: 0.3 -> 0.3302
- rule via_min_size: 0.4 -> 0.6858
