File: kicad/buspirate-breadboard-connector.sch (KiCad schematic (older format))
At the start: 2 parts

Commit message: minor changes to the footprints and creation of gerbers
Parts:
- BP1: footprint Pin_Headers:Pin_Header_Straight_2x05 -> breadboard-connector:header_2x5
Changed lines of the file:
@@
 LIBS:valves
 LIBS:buspirate
+LIBS:buspirate-breadboard-connector-cache
 EELAYER 25 0
 EELAYER END
@@
 F 0 "BP1" H 6050 2850 60  0000 C CNN
 F 1 "BusPirate" H 5650 3550 60  0000 C CNN
-F 2 "Pin_Headers:Pin_Header_Straight_2x05" H 5650 3000 60  0001 C CNN
+F 2 "breadboard-connector:header_2x5" H 5650 3000 60  0001 C CNN
 F 3 "" H 5650 3000 60  0000 C CNN
 	1    5650 3000
